Commit message: add lidar sensors. watch summit_description -> urdf -> base ->summit_base urdf xarco

File: for_mad/src/summit_description/robot/summit.urdf.xacro (robot description, xacro)
@@ -8,5 +8,4 @@
 	<xacro:include filename="$(find summit_description)/urdf/base/summit_base.urdf.xacro" />
 	<xacro:include filename="$(find summit_description)/urdf/base/summit_base.gazebo.xacro" />
-	<!--<xacro:include filename="$(find realsense2_description)/urdf/_d435.urdf.xacro" />-->
 	<!-- Wheel parameters -->
 	<xacro:property name="wheel_offset_x" value="0.19" />    <!-- x,y,z in translation from base_link to the center of the wheel 		standart=0.2225-->
@@ -28,357 +27,6 @@
 		</xacro:omni_wheel>
 		<xacro:omni_steering/>
-		<!-- REALSENSE CAMERA -->
-  <!--<xacro:if value="$(arg realsense_enable)">
-    <xacro:sensor_d435 name="realsense_d435" topics_ns="realsense_d435" parent="base_link" publish_pointcloud="$(arg pointcloud_enable)" >
-      <origin xyz="0.077 0 0" rpy="0 0 0" />
-    </xacro:sensor_d435>
-  </xacro:if>-->
    		<!-- MANIPULATOR, PLEASE, CREATE A XACRO MACRO -->
-		<joint name="ang_base" type="fixed">
-		<parent link="summit_base_link"/>
-		<child link="ang_link0"/>
-		<origin rpy = "0 0 -1.57" xyz="-0.16 0 0.05" />
-	</joint>
-	<link name="ang_link0">
-		<visual>
-			<geometry>
-				<mesh filename="package://angle_arm_model_gazebo/meshes/link1.dae" scale="0.001 0.001 0.001"/>
-			</geometry>
-		</visual>
-		<inertial>
-			<origin xyz="0 0 0.5" rpy="0 0 0"/>
-			<mass value="1"/>
-			<inertia
-				ixx="0.01" ixy="0.0" ixz="0.0"
-				iyy="0.01" iyz="0.0"
-				izz="0.01"/>
-		</inertial>
-	</link>
-	<joint name="ang_joint1" type="continuous">
-		<parent link="ang_link0"/>
-		<child link="ang_link1"/>
-		<origin xyz = "0 0 0.117" rpy="1.57 0 -1.57" />
-		<axis xyz="0 1 0" />
-		<dynamics damping="0.99"/>
-		<limit effort="5.0" velocity="5.0"/>
-	</joint>
-	<link name="ang_link1">
-		<visual>
-			<geometry>
-				<mesh filename="package://angle_arm_model_gazebo/meshes/link2.dae" scale="0.001 0.001 0.001"/>
-			</geometry>
-		</visual>
-		<inertial>
-			<origin xyz="0 0.25 0" rpy="0 0 0"/>
-			<mass value="0.001"/>
-			<inertia
-				ixx="0.01" ixy="0.0" ixz="0.0"
-				iyy="0.01" iyz="0.0"
-				izz="0.01"/>
-		</inertial>
-	</link>
-	<joint name="ang_joint2" type="continuous">
-		<parent link="ang_link1"/>
-		<child link="ang_link2"/>
-		<origin xyz = "0 0.0518 0" rpy="0 0 0" />
-		<axis xyz="0 0 1" />
-		<dynamics damping="0.99"/>
-		<limit effort="5.0" velocity="5.0"/>
-	</joint>
-	<link name="ang_link2">
-		<visual>
-			<geometry>
-				<mesh filename="package://angle_arm_model_gazebo/meshes/link3.dae" scale="0.001 0.001 0.001"/>
-			</geometry>
-		</visual>
-		<inertial>
-			<origin xyz="0 0.15 0" rpy="0 0 0"/>
-			<mass value="0.001"/>
-			<inertia
-				ixx="0.01" ixy="0.0" ixz="0.0"
-				iyy="0.01" iyz="0.0"
-				izz="0.01"/>
-		</inertial>
-	</link>
-	<joint name="ang_joint3" type="continuous">
-		<parent link="ang_link2"/>
-		<child link="ang_link3"/>
-		<origin xyz = "0.0626 0.1989 0" rpy="0 0 0" />
-		<axis xyz="0 0 1" />
-		<dynamics damping="0.99"/>
-		<limit effort="5.0" velocity="5.0"/>
-	</joint>
-	<link name="ang_link3">
-		<visual>
-			<geometry>
-				<mesh filename="package://angle_arm_model_gazebo/meshes/link4.dae" scale="0.001 0.001 0.001"/>
-			</geometry>
-		</visual>
-		<inertial>
-			<origin xyz="0 0 0" rpy="0 0 0"/>
-			<mass value="0.001"/>
-			<inertia
-				ixx="0.01" ixy="0.0" ixz="0.0"
-				iyy="0.01" iyz="0.0"
-				izz="0.01"/>
-		</inertial>
-	</link>
-	<joint name="ang_joint4" type="continuous">
-		<parent link="ang_link3"/>
-		<child link="ang_link4"/>
-		<origin xyz = "0.13093 0 0" rpy="-1.57 0 1.57" />
-		<axis xyz="0 -1 0" />
-		<dynamics damping="0.99"/>
-		<limit effort="5.0" velocity="5.0"/>
-	</joint>
-	<link name="ang_link4">
-		<visual>
-			<geometry>
-				<mesh filename="package://angle_arm_model_gazebo/meshes/link5.dae" scale="0.001 0.001 0.001"/>
-			</geometry>
-		</visual>
-		<inertial>
-			<origin xyz="0 0 0" rpy="0 0 0"/>
-			<mass value="0.001"/>
-			<inertia
-				ixx="0.01" ixy="0.0" ixz="0.0"
-				iyy="0.01" iyz="0.0"
-				izz="0.01"/>
-		</inertial>
-	</link>
-	<joint name="ang_joint5" type="continuous">
-		<parent link="ang_link4"/>
-		<child link="ang_link5"/>
-		<origin xyz = "0 0 -0.06174" rpy="0 0 0" />
-		<axis xyz="0 0 -1" />
-		<dynamics damping="0.99"/>
-		<limit effort="5.0" velocity="5.0"/>
-	</joint>
-	<link name="ang_link5">
-		<visual>
-			<geometry>
-				<mesh filename="package://angle_arm_model_gazebo/meshes/link6.dae" scale="0.001 0.001 0.001"/>
-			</geometry>
-		</visual>
-		<inertial>
-			<origin xyz="0 0 0" rpy="0 0 0"/>
-			<mass value="0.001"/>
-			<inertia
-				ixx="0.01" ixy="0.0" ixz="0.0"
-				iyy="0.01" iyz="0.0"
-				izz="0.01"/>
-		</inertial>
-	</link>
-<!--	<xacro:sensor_d435 name="sensor_d435" topics_ns="sensor_d435" parent="ang_link5">
-    <origin rpy="0 1.625 0" xyz="0.019 0 -0.0555"/>
-  </xacro:sensor_d435> -->
-<!--
-  <link name="cam_on_manipulator">
-  	<inertial>
-  		<mass value="0.00001" />
-  		<inertia
-				ixx="0.01" ixy="0.0" ixz="0.0"
-				iyy="0.01" iyz="0.0"
-				izz="0.01"/>
-  	</inertial>
-  	<visual>
-  		<origin rpy="0 0 0" xyz="0 0 0" />
-  		<geometry>
-  			<box size="0.01 0.01 0.01" />
-  		</geometry>
-  	</visual>
-  </link>
-  <joint name="fixed_cam" type="fixed">
-  	<parent link="ang_link5" />
-  	<child link="cam_on_manipulator" />
-  	<origin rpy="0 1.625 0" xyz="0.019 0 -0.0555"/>
-  	<dynamics damping="0.99"/>
-  	<limit effort="5.0" velocity="5.0"/>
-  </joint> -->
-  <xacro:sensor_d435 name="sensor_d435" topics_ns="sensor_d435" parent="ang_link5">
-    <origin rpy="0 1.625 0" xyz="0.019 0 -0.0555"/>
-  </xacro:sensor_d435>
-  <!-- why i wrote this... -->
-  <!--<joint name="cam_connector">
-  		<parent link="ang_link5" />
-  		<child link="sensor_d435" />
-  		<axis xyz="0 0 1" />
-		<limit effort="3" lower="0" upper="0.025" velocity="0.05"/>
-		<dynamics damping="0.99"/>
-  </joint> -->
-	<joint name="ang_gripper" type="prismatic">
-		<parent link="ang_link5"/>
-		<child link="ang_link6"/>
-		<origin xyz = "0 0 -0.0715" rpy="1.57 3.14 0" />
-		<axis xyz="0 0 1" />
-		<limit effort="3" lower="0" upper="0.025" velocity="0.05"/>
-		<dynamics damping="0.99"/>
-	</joint>
-	<link name="ang_link6">
-		<collision>
-			<geometry>
-				<mesh filename="package://angle_arm_model_gazebo/meshes/link7.dae" scale="0.001 0.001 0.001"/>
-			</geometry>
-		</collision>
-		<visual>
-			<geometry>
-				<mesh filename="package://angle_arm_model_gazebo/meshes/link7.dae" scale="0.001 0.001 0.001"/>
-			</geometry>
-		</visual>
-		<inertial>
-			<origin xyz="0 0 0" rpy="0 0 0"/>
-			<mass value="0.001"/>
-			<inertia
-				ixx="0.01" ixy="0.0" ixz="0.0"
-				iyy="0.01" iyz="0.0"
-				izz="0.01"/>
-		</inertial>
-	</link>
-	<joint name="ang_gripper_sub" type="prismatic">
-		<parent link="ang_link5"/>
-		<child link="ang_link7"/>
-		<origin xyz = "0 0 -0.0715" rpy="-1.57 0 0" />
-		<axis xyz="0 0 1" />
-		<limit effort="3" lower="0" upper="0.025" velocity="0.05"/>
-	        <mimic joint="ang_gripper" multiplier="1" offset="0"/>
-		<dynamics damping="0.99"/>
-	</joint>
-	<link name="ang_link7">
-		<collision>
-			<geometry>
-				<mesh filename="package://angle_arm_model_gazebo/meshes/link7.dae" scale="0.001 0.001 0.001"/>
-			</geometry>
-		</collision>
-		<visual>
-			<geometry>
-				<mesh filename="package://angle_arm_model_gazebo/meshes/link7.dae" scale="0.001 0.001 0.001"/>
-			</geometry>
-		</visual>
-		<inertial>
-			<origin xyz="0 0 0" rpy="0 0 0"/>
-			<mass value="0.001"/>
-			<inertia
-				ixx="0.01" ixy="0.0" ixz="0.0"
-				iyy="0.01" iyz="0.0"
-				izz="0.01"/>
-		</inertial>
-	</link>
-<!-- transmission -->
-	<transmission name="ang_tran1">
-		<type>transmission_interface/SimpleTransmission</type>
-		<joint name="ang_joint1">
-			<hardwareInterface>hardware_interface/EffortJointInterface</hardwareInterface>
-		</joint>
-		<actuator name="ang_motor1">
-			<hardwareInterface>hardware_interface/EffortJointInterface</hardwareInterface>
-			<mechanicalReduction>1</mechanicalReduction>
-		</actuator>
-	</transmission>
-	<transmission name="ang_tran2">
-		<type>transmission_interface/SimpleTransmission</type>
-		<joint name="ang_joint2">
-			<hardwareInterface>hardware_interface/EffortJointInterface</hardwareInterface>
-		</joint>
-		<actuator name="ang_motor2">
-			<hardwareInterface>hardware_interface/EffortJointInterfacee</hardwareInterface>
-			<mechanicalReduction>1</mechanicalReduction>
-		</actuator>
-	</transmission>
-	<transmission name="ang_tran3">
-		<type>transmission_interface/SimpleTransmission</type>
-		<joint name="ang_joint3">
-			<hardwareInterface>hardware_interface/EffortJointInterface</hardwareInterface>
-		</joint>
-		<actuator name="ang_motor3">
-			<hardwareInterface>hardware_interface/EffortJointInterfacee</hardwareInterface>
-			<mechanicalReduction>1</mechanicalReduction>
-		</actuator>
-	</transmission>
-	<transmission name="ang_tran4">
-		<type>transmission_interface/SimpleTransmission</type>
-		<joint name="ang_joint4">
-			<hardwareInterface>hardware_interface/EffortJointInterface</hardwareInterface>
-		</joint>
-		<actuator name="ang_motor4">
-			<hardwareInterface>hardware_interface/EffortJointInterfacee</hardwareInterface>
-			<mechanicalReduction>1</mechanicalReduction>
-		</actuator>
-	</transmission>
-	<transmission name="ang_tran5">
-		<type>transmission_interface/SimpleTransmission</type>
-		<joint name="ang_joint5">
-			<hardwareInterface>hardware_interface/EffortJointInterface</hardwareInterface>
-		</joint>
-		<actuator name="ang_motor5">
-			<hardwareInterface>hardware_interface/EffortJointInterfacee</hardwareInterface>
-			<mechanicalReduction>1</mechanicalReduction>
-		</actuator>
-	</transmission>
-	<transmission name="ang_tran5">
-		<type>transmission_interface/SimpleTransmission</type>
-		<joint name="ang_gripper">
-			<hardwareInterface>hardware_interface/EffortJointInterface</hardwareInterface>
-		</joint>
-		<actuator name="ang_motor5">
-			<hardwareInterface>hardware_interface/EffortJointInterfacee</hardwareInterface>
-			<mechanicalReduction>1</mechanicalReduction>
-		</actuator>
-	</transmission>
-	<transmission name="ang_tran5">
-		<type>transmission_interface/SimpleTransmission</type>
-		<joint name="ang_gripper">
-			<hardwareInterface>hardware_interface/EffortJointInterface</hardwareInterface>
-		</joint>
-		<actuator name="ang_motor5">
-			<hardwareInterface>hardware_interface/EffortJointInterfacee</hardwareInterface>
-			<mechanicalReduction>1</mechanicalReduction>
-		</actuator>
-	</transmission>
-	<transmission name="ang_tran5">
-		<type>transmission_interface/SimpleTransmission</type>
-		<joint name="ang_gripper_sub">
-			<hardwareInterface>hardware_interface/EffortJointInterface</hardwareInterface>
-		</joint>
-		<actuator name="ang_motor5">
-			<hardwareInterface>hardware_interface/EffortJointInterfacee</hardwareInterface>
-			<mechanicalReduction>1</mechanicalReduction>
-		</actuator>
-	</transmission>
-  <gazebo reference="ang_link0">
-    <material>Gazebo/Gray</material>
-  </gazebo>
-  <gazebo reference="ang_link1">
-    <material>Gazebo/Gray</material>
-  </gazebo>
-  <gazebo reference="ang_link2">
-    <material>Gazebo/Gray</material>
-  </gazebo>
-  <gazebo reference="ang_link3">
-    <material>Gazebo/Gray</material>
-  </gazebo>
-  <gazebo reference="ang_link4">
-    <material>Gazebo/Gray</material>
-  </gazebo>
-  <gazebo reference="ang_link5">
-    <material>Gazebo/Gray</material>
-  </gazebo>
-  <gazebo reference="ang_link7">
-    <material>Gazebo/Orange</material>
-        <kp>10000.0</kp>
-        <kd>10000.0</kd>
-        <mu1>1000.0</mu1>
-        <mu2>1000.0</mu2>
-    <minDepth>0.001</minDepth>
-    <maxVel>0</maxVel>
-  </gazebo>
-  <gazebo reference="ang_link6">
-        <kp>10000.0</kp>
-        <kd>10000.0</kd>
-        <mu1>1000.0</mu1>
-        <mu2>1000.0</mu2>
-    <minDepth>0.001</minDepth>
-    <maxVel>0</maxVel>
-    <material>Gazebo/Orange</material>
-  </gazebo>
+	<xacro:include filename="$(find summit_description)/robot/m.gazabo.xacro" />
   <!-- MANIPULATOR, PLEASE, CREATE A XACRO MACRO -->
    </xacro:macro>

File: for_mad/src/summit_description/urdf/base/summit_base.gazebo.xacro (robot description, xacro)
@@ -4,4 +4,5 @@
 		<gazebo>
     	<plugin name="object_controller" filename="libgazebo_ros_planar_move.so">
+    	<robotNamespace>/base</robotNamespace>
       	<commandTopic>cmd_vel</commandTopic>
       	<odometryTopic>odom</odometryTopic>

File: for_mad/src/summit_description/urdf/base/summit_base.urdf.xacro (robot description, xacro)
@@ -48,4 +48,165 @@
     </collision>
   </link>
+  <!-- ******************************************HOKUYO LIDAR ******************************-->
+  <joint name="hokuyo_joint" type="fixed">
+        <axis xyz="0 0 0" />
+        <origin xyz="-0.29 0 0.07" rpy="0 0 3.14"/>
+        <parent link="summit_base_footprint"/>
+        <child link="hokuyo_link"/>
+    </joint>
+  <!-- Hokuyo Laser -->
+ <link name="hokuyo_link">
+        <collision>
+          <origin xyz="0 0 0" rpy="0 0 0"/>
+          <geometry>
+        <box size="0.1 0.1 0.1"/>
+          </geometry>
+        </collision>
+        <visual>
+          <origin xyz="0 0 0" rpy="0 0 0"/>
+          <geometry>
+            <mesh filename="package://summit_description/meshes/hokuyo.dae"/>
+          </geometry>
+        </visual>
+        <inertial>
+          <mass value="1e-5" />
+          <origin xyz="0 0 0" rpy="0 0 0"/>
+          <inertia ixx="1e-6" ixy="0" ixz="0" iyy="1e-6" iyz="0" izz="1e-6" />
+        </inertial>
+  </link>
+  <!--<gazebo reference="hokuyo_link">
+    <sensor type="gpu_ray" name="head_hokuyo_sensor">
+      <pose>0 0 0 0 0 0</pose>
+      <visualize>false</visualize>
+      <update_rate>40</update_rate>
+      <ray>
+        <scan>
+          <horizontal>
+            <samples>720</samples>
+            <resolution>1</resolution>
+            <min_angle>-1.570796</min_angle>
+            <max_angle>1.570796</max_angle>
+          </horizontal>
+        </scan>
+        <range>
+          <min>0.10</min>
+          <max>30.0</max>
+          <resolution>0.01</resolution>
+        </range>
+        <noise>
+          <type>gaussian</type>-->
+          <!-- Noise parameters based on published spec for Hokuyo laser
+               achieving "+-30mm" accuracy at range < 10m.  A mean of 0.0m and
+               stddev of 0.01m will put 99.7% of samples within 0.03m of the true
+               reading.-->
+     <!--     <mean>0.0</mean>
+          <stddev>0.01</stddev>
+        </noise>
+      </ray>
+      <plugin name="gazebo_ros_head_hokuyo_controller" filename="libgazebo_ros_gpu_laser.so">
+        <topicName>/summit_description/laser/scan</topicName>
+        <frameName>hokuyo_link</frameName>
+      </plugin>
+    </sensor>
+  </gazebo> -->
+  <gazebo reference="hokuyo_link">
+    <sensor type="ray" name="head_hokuyo_sensor">
+      <pose>0 0 0 0 0 0</pose>
+      <visualize>true</visualize>
+      <update_rate>40</update_rate>
+      <ray>
+        <scan>
+          <horizontal>
+            <samples>720</samples>
+            <resolution>1</resolution>
+            <min_angle>-1.570796</min_angle>
+            <max_angle>1.570796</max_angle>
+          </horizontal>
+        </scan>
+        <range>
+          <min>0.10</min>
+          <max>30.0</max>
+          <resolution>0.01</resolution>
+        </range>
+        <noise>
+          <type>gaussian</type>
+          <!-- Noise parameters based on published spec for Hokuyo laser
+               achieving "+-30mm" accuracy at range < 10m.  A mean of 0.0m and
+               stddev of 0.01m will put 99.7% of samples within 0.03m of the true
+               reading. -->
+          <mean>0.0</mean>
+          <stddev>0.01</stddev>
+        </noise>
+      </ray>
+      <plugin name="gazebo_ros_head_hokuyo_controller" filename="libgazebo_ros_laser.so">
+        <topicName>/scan</topicName>
+        <frameName>hokuyo_link</frameName>
+      </plugin>
+    </sensor>
+  </gazebo>
+  <!-- ******************************************HOKUYO LIDAR ******************************-->
+  <!-- ******************************************RPLIDAR******************************-->
+  <joint name="rplidar_joint" type="fixed">
+        <axis xyz="0 0 0" />
+        <origin xyz="0.204590 0 0.161790" rpy="0 0 0"/>
+        <parent link="summit_base_footprint"/>
+        <child link="rplidar_link"/>
+    </joint>
+  <!-- RPLIDAR Laser -->
+ <link name="rplidar_link">
+        <visual>
+          <origin xyz="0 0 0" rpy="0 0 0"/>
+          <geometry>
+              <box size="0.01 0.01 0.01"/>
+                <!-- NO GOD PLEASE NO!!!!!!!!!!!!!!!!!!!!!!!!!!!!!!!!!!!!!!!!!!!!!!!!!!!!!!!!!!!!!!!!!!!!!!!!!!!!!!!!!!!!!!!!!!!! -->
+         <!--   <mesh filename="package://summit_description/meshes/laser/lds.stl" scale="0.001 0.001 0.001"/> -->
+          </geometry>
+        </visual>
+        <collision>
+          <origin xyz="0.015 0 -0.0065" rpy="0 0 0"/>
+          <geometry>
+              <cylinder length="0.0315" radius="0.055"/>
+          </geometry>
+        </collision>
+        <inertial>
+          <mass value="0.114" />
+          <origin xyz="0 0 0" />
+          <inertia ixx="0.001" ixy="0.0" ixz="0.0"
+                   iyy="0.001" iyz="0.0"
+                   izz="0.001" />
+        </inertial>
+  </link>
+  <gazebo reference="rplidar_link">
+    <sensor type="ray" name="head_rplidar_sensor">
+      <pose>0 0 0 0 0 0</pose>
+      <visualize>true</visualize>
+      <update_rate>5</update_rate>
+      <ray>
+        <scan>
+            <horizontal>
+              <samples>720</samples>
+              <resolution>1</resolution>
+              <min_angle>-1.570796</min_angle>
+              <max_angle>1.570796</max_angle>
+            </horizontal>
+        </scan>
+        <range>
+            <min>0.120</min>
+            <max>3.5</max>
+            <resolution>0.015</resolution>
+        </range>
+        <noise>
+          <type>gaussian</type>
+          <mean>0.0</mean>
+          <stddev>0.01</stddev>
+        </noise>
+      </ray>
+      <plugin name="gazebo_ros_head_hokuyo_controller" filename="libgazebo_ros_laser.so">
+        <topicName>/scan_two</topicName>
+        <frameName>rplidar_link</frameName>
+      </plugin>
+    </sensor>
+  </gazebo>
+  <!-- ****************************************** RPLIDAR******************************-->
   </xacro:macro>
 </robot>

File: for_mad/src/summit_description/urdf/wheels/omni_wheel.urdf.xacro (robot description, xacro)
@@ -46,5 +46,5 @@
       </inertial>
     </link>
-    <!-- Transmission is important to link the joints and the controller (see summit_xl_control/config/summit_xl_control.yaml)-->
+    <!-- Transmission is important to link the joints and the controller (see summit_xl_control/config/summit_xl_control.yaml)
     <transmission name="${prefix}_wheel_joint_trans">
       <type>transmission_interface/SimpleTransmission</type>
@@ -56,4 +56,5 @@
       </actuator>
     </transmission>
+-->
     <gazebo reference="${prefix}_wheel_link">
 		<mu1 value="1.0"/>
